Commit message: Add torque_limits YAML pipeline and retune PD gains for SNU deployment
- pd_gains.yaml: new torque_limits section (all 0.8, normalized duty),
  overriding the driver's hardcoded default_torque_limit_table
- ros2_control xacro (single/dual): pass torque_joint** hardware params
- ros_utility.cpp: parse torque_ params into torque_limit_table_,
  falling back to hardcoded defaults when absent
- pd_gains.yaml: per-joint differential PD gains (Kp 1.5-3.0,
  Kd 0.095-0.14) tuned from 100 Hz replay analysis
- COLCON_IGNORE for unused gazebo plugin and plexus hardware packages
- LOCAL_CHANGES.md: document all deviations from upstream

Co-Authored-By: Claude Fable 5 <noreply@anthropic.com>

File: allegro_hand_bringup/config/v4/dual_hand/allegro_hand.ros2_control.xacro (robot description, xacro)
@@ -5,4 +5,5 @@
         <xacro:property name="p_gains" value="${xacro.load_yaml(pd_gains_file)['p_gains']}"/>
         <xacro:property name="d_gains" value="${xacro.load_yaml(pd_gains_file)['d_gains']}"/>
+        <xacro:property name="torque_limits" value="${xacro.load_yaml(pd_gains_file)['torque_limits']}"/>
         <ros2_control name="${name}" type="system">
             <hardware>
@@ -50,4 +51,20 @@
                     <param name="d_joint32">${d_gains['joint32']}</param>
                     <param name="d_joint33">${d_gains['joint33']}</param>
+                    <param name="torque_joint00">${torque_limits['joint00']}</param>
+                    <param name="torque_joint01">${torque_limits['joint01']}</param>
+                    <param name="torque_joint02">${torque_limits['joint02']}</param>
+                    <param name="torque_joint03">${torque_limits['joint03']}</param>
+                    <param name="torque_joint10">${torque_limits['joint10']}</param>
+                    <param name="torque_joint11">${torque_limits['joint11']}</param>
+                    <param name="torque_joint12">${torque_limits['joint12']}</param>
+                    <param name="torque_joint13">${torque_limits['joint13']}</param>
+                    <param name="torque_joint20">${torque_limits['joint20']}</param>
+                    <param name="torque_joint21">${torque_limits['joint21']}</param>
+                    <param name="torque_joint22">${torque_limits['joint22']}</param>
+                    <param name="torque_joint23">${torque_limits['joint23']}</param>
+                    <param name="torque_joint30">${torque_limits['joint30']}</param>
+                    <param name="torque_joint31">${torque_limits['joint31']}</param>
+                    <param name="torque_joint32">${torque_limits['joint32']}</param>
+                    <param name="torque_joint33">${torque_limits['joint33']}</param>
                 </xacro:if>
             </hardware>

File: allegro_hand_bringup/config/v4/single_hand/allegro_hand.ros2_control.xacro (robot description, xacro)
@@ -5,4 +5,5 @@
         <xacro:property name="p_gains" value="${xacro.load_yaml(pd_gains_file)['p_gains']}"/>
         <xacro:property name="d_gains" value="${xacro.load_yaml(pd_gains_file)['d_gains']}"/>
+        <xacro:property name="torque_limits" value="${xacro.load_yaml(pd_gains_file)['torque_limits']}"/>
         <ros2_control name="${name}" type="system">
             <hardware>
@@ -50,4 +51,20 @@
                     <param name="d_joint32">${d_gains['joint32']}</param>
                     <param name="d_joint33">${d_gains['joint33']}</param>
+                    <param name="torque_joint00">${torque_limits['joint00']}</param>
+                    <param name="torque_joint01">${torque_limits['joint01']}</param>
+                    <param name="torque_joint02">${torque_limits['joint02']}</param>
+                    <param name="torque_joint03">${torque_limits['joint03']}</param>
+                    <param name="torque_joint10">${torque_limits['joint10']}</param>
+                    <param name="torque_joint11">${torque_limits['joint11']}</param>
+                    <param name="torque_joint12">${torque_limits['joint12']}</param>
+                    <param name="torque_joint13">${torque_limits['joint13']}</param>
+                    <param name="torque_joint20">${torque_limits['joint20']}</param>
+                    <param name="torque_joint21">${torque_limits['joint21']}</param>
+                    <param name="torque_joint22">${torque_limits['joint22']}</param>
+                    <param name="torque_joint23">${torque_limits['joint23']}</param>
+                    <param name="torque_joint30">${torque_limits['joint30']}</param>
+                    <param name="torque_joint31">${torque_limits['joint31']}</param>
+                    <param name="torque_joint32">${torque_limits['joint32']}</param>
+                    <param name="torque_joint33">${torque_limits['joint33']}</param>
                 </xacro:if>
             </hardware>
